Commit message: updated basic version

File: src/robostore_bringup/urdf/table.urdf.xacro (robot description, xacro)
@@ -18,5 +18,7 @@
           <box size="${table_width} ${table_depth} ${table_height}"/>
         </geometry>
-        <material name="white"/>
+        <material name="">
+          <color rgba="0.6 0.1960 0.8 1" />
+        </material>
       </visual>
       <collision>
