Commit message: updated platform

File: src/robostore_bringup/urdf/dual_arm_robot_16w_env.urdf.xacro (robot description, xacro)
@@ -30,5 +30,5 @@
   </xacro:dual_arm_robot>
   <xacro:table name="table" id="1" parent="map">
-    <origin xyz="1.47 0.8 0" rpy="0 0 3.14159265359"/>
+    <origin xyz="1.38 0.8 0" rpy="0 0 3.14159265359"/>
   </xacro:table>
   <xacro:rack name="rack" id="1" parent="map">

File: src/robostore_bringup/urdf/table.urdf.xacro (robot description, xacro)
@@ -30,20 +30,20 @@
     </link>
     <xacro:place_location parent="${name}_${id}_base_link" prefix="${name}_${id}" index="1">
-      <origin xyz="0.4 0.15 ${table_height}" rpy="0 0 0"/>
+      <origin xyz="0.45 0.15 ${table_height}" rpy="0 0 0"/>
     </xacro:place_location>
     <xacro:place_location parent="${name}_${id}_base_link" prefix="${name}_${id}" index="2">
-      <origin xyz="0.55 0.15 ${table_height}" rpy="0 0 0"/>
+      <origin xyz="0.6 0.15 ${table_height}" rpy="0 0 0"/>
     </xacro:place_location>
     <xacro:place_location parent="${name}_${id}_base_link" prefix="${name}_${id}" index="3">
-      <origin xyz="0.7 0.15 ${table_height}" rpy="0 0 0"/>
+      <origin xyz="0.75 0.15 ${table_height}" rpy="0 0 0"/>
     </xacro:place_location>
     <xacro:place_location parent="${name}_${id}_base_link" prefix="${name}_${id}" index="4">
-      <origin xyz="0.4 0.05 ${table_height}" rpy="0 0 0"/>
+      <origin xyz="0.45 0.05 ${table_height}" rpy="0 0 0"/>
     </xacro:place_location>
     <xacro:place_location parent="${name}_${id}_base_link" prefix="${name}_${id}" index="5">
-      <origin xyz="0.55 0.05 ${table_height}" rpy="0 0 0"/>
+      <origin xyz="0.6 0.05 ${table_height}" rpy="0 0 0"/>
     </xacro:place_location>
     <xacro:place_location parent="${name}_${id}_base_link" prefix="${name}_${id}" index="6">
-      <origin xyz="0.7 0.05 ${table_height}" rpy="0 0 0"/>
+      <origin xyz="0.75 0.05 ${table_height}" rpy="0 0 0"/>
     </xacro:place_location>
   </xacro:macro>
