Commit message: added new controller

File: src/robostore_bringup/urdf/dual_arm_in_table.urdf.xacro (robot description, xacro)
@@ -16,5 +16,5 @@
     <xacro:property name="M_PI" value="3.14159265359" />
     <xacro:property name="M_PI_2" value="1.57079632679" />
-    <xacro:include filename="$(find dual_arm_description)/urdf/dual_arm.urdf.xacro" />
+    <xacro:include filename="$(find dual_arm_description)/urdf/dual_arm_w_mdh.urdf.xacro" />
     <xacro:include filename="$(find dual_arm_configure)/config/dual_arm.ros2_control.xacro" />
     <xacro:include filename="$(find dual_arm_robot)/robot_model/left_eef.urdf.xacro" />
@@ -26,5 +26,5 @@
     <xacro:arg name="to_be_done" default="false"/>
     <xacro:dual_arm name="dual_arm" parent="${parent}">
-      <origin xyz="-0.0064 0 0.26" rpy="0 0 ${M_PI}"/>
+      <origin xyz="0 0 0" rpy="0 0 0"/>
     </xacro:dual_arm>
     <xacro:dual_arm_ros2_control
@@ -41,5 +41,5 @@
     </xacro:sensor_d435>
     <xacro:left_eef name="${left_eef_name}" parent="link7_left">
-      <origin xyz="0 0.0335 0" rpy="0 0 0"/>
+      <origin xyz="0.0335 0 0" rpy="0 0 ${-M_PI_2}"/>
     </xacro:left_eef>
     <xacro:sensor_d435
@@ -50,5 +50,5 @@
     </xacro:sensor_d435>
     <xacro:right_eef name="${right_eef_name}" parent="link7_right">
-      <origin xyz="0 0.0335 0" rpy="0 ${M_PI} 0"/>
+      <origin xyz="0.0335 0 0" rpy="0 0 ${-M_PI_2}"/>
     </xacro:right_eef>
   </xacro:macro>
@@ -69,5 +69,5 @@
       <origin xyz="0 0 0.395" rpy="0 0 0"/>
       <geometry>
-        <box size="0.6 0.6 0.79"/>
+        <box size="0.5 0.5 0.79"/>
       </geometry>
       <material name="">
@@ -78,10 +78,10 @@
       <origin xyz="0 0 0.395" rpy="0 0 0"/>
       <geometry>
-        <box size="0.6 0.6 0.79"/>
+        <box size="0.5 0.5 0.79"/>
       </geometry>
     </collision>
   </link>
   <joint name="dual_arm_robot_base_joint" type="fixed">
-    <origin xyz="0.215 0.215 0.80" rpy="0 0 0.5235987756"/>
+    <origin xyz="0 0 0.805" rpy="0 0 0"/>
     <parent link="table_base_link"/>
     <child link="dual_arm_base_link"/>

Commit message: added chrt

File: src/robostore_bringup/urdf/dual_arm_in_table.urdf.xacro (robot description, xacro)
@@ -6,4 +6,6 @@
   <xacro:arg name="right_arm_sim" default="true" />
   <xacro:arg name="right_arm_can_interface" default="can1" />
+  <xacro:property name="M_PI" value="3.14159265359" />
+  <xacro:property name="M_PI_2" value="1.57079632679" />
   <xacro:macro name="dual_arm_in_table" params="
     name
@@ -83,5 +85,5 @@
   </link>
   <joint name="dual_arm_robot_base_joint" type="fixed">
-    <origin xyz="0 0 0.805" rpy="0 0 0"/>
+    <origin xyz="0.1 0 0.805" rpy="0 0 0"/>
     <parent link="table_base_link"/>
     <child link="dual_arm_base_link"/>
@@ -97,3 +99,69 @@
     <origin xyz="0 0 0" rpy="0 0 0"/>
   </xacro:dual_arm_in_table>
+  <!-- <link name="box_table_base_link">
+    <visual>
+      <origin xyz="0 0 0.3175" rpy="0 0 0"/>
+      <geometry>
+        <box size="0.73 0.5 0.635"/>
+      </geometry>
+      <material name="">
+        <color rgba="0.95 0.95 0.95 1" />
+      </material>
+    </visual>
+    <collision>
+      <origin xyz="0 0 0.3175" rpy="0 0 0"/>
+      <geometry>
+        <box size="0.73 0.5 0.635"/>
+      </geometry>
+    </collision>
+  </link>
+  <joint name="box_table_joint" type="fixed">
+    <origin xyz="0.625 0 0" rpy="0 0 0"/>
+    <parent link="table_base_link"/>
+    <child link="box_table_base_link"/>
+  </joint>
+  <link name="box_in_link">
+    <visual>
+      <origin xyz="0 0 0" rpy="0 0 0"/>
+      <geometry>
+        <mesh filename="package://robostore_bringup/meshes/visual/material_box.STL" />
+      </geometry>
+      <material name="">
+        <color rgba="0.15 0.15 0.15 1" />
+      </material>
+    </visual>
+    <collision>
+      <origin xyz="0 0 0" rpy="0 0 0"/>
+      <geometry>
+        <mesh filename="package://robostore_bringup/meshes/visual/material_box.STL" />
+      </geometry>
+    </collision>
+  </link>
+  <joint name="box_in_joint" type="fixed">
+    <origin xyz="-0.355 0.245 0.635" rpy="0 0 -${M_PI_2}"/>
+    <parent link="box_table_base_link"/>
+    <child link="box_in_link"/>
+  </joint>
+  <link name="box_out_link">
+    <visual>
+      <origin xyz="0 0 0" rpy="0 0 0"/>
+      <geometry>
+        <mesh filename="package://robostore_bringup/meshes/visual/material_box.STL" />
+      </geometry>
+      <material name="">
+        <color rgba="0.15 0.15 0.15 1" />
+      </material>
+    </visual>
+    <collision>
+      <origin xyz="0 0 0" rpy="0 0 0"/>
+      <geometry>
+        <mesh filename="package://robostore_bringup/meshes/visual/material_box.STL" />
+      </geometry>
+    </collision>
+  </link>
+  <joint name="box_out_joint" type="fixed">
+    <origin xyz="0 0.245 0.635" rpy="0 0 -${M_PI_2}"/>
+    <parent link="box_table_base_link"/>
+    <child link="box_out_link"/>
+  </joint> -->
 </robot>
