Commit message: updated basic version

File: src/fold_elevator/fold_elevator_configure/config/fold_elevator.ros2_control.xacro (robot description, xacro)
@@ -1,80 +1,81 @@
 <?xml version="1.0"?>
 <robot xmlns:xacro="http://www.ros.org/wiki/xacro">
-    <xacro:macro name="fold_elevator_ros2_control" params="name sim can_interface">
-        <ros2_control name="fold_elevator" type="system">
-            <hardware>
-                <xacro:if value="${sim}">
-                    <plugin>mock_components/GenericSystem</plugin>
-                </xacro:if>
-                <xacro:unless value="${sim}">
-                    <plugin>fold_elevator_hardware_interface/FoldElevatorHardwareInterface</plugin>
-                    <param name="can_interface">${can_interface}</param>
-                </xacro:unless>
-            </hardware>
-            <joint name="joint1">
-                <command_interface name="position"/>
-                <state_interface name="position"/>
-                <state_interface name="velocity"/>
-                <param name="can_id">0x60</param>
-                <param name="gear_ratio">101.0</param>
-                <param name="position_offset">A0CC</param>
-                <param name="max_current">22000</param>
-                <param name="min_current">-22000</param>
-                <param name="position_p">5000</param>
-                <param name="position_d">450</param>
-                <param name="velocity_p">550</param>
-                <param name="velocity_i">250</param>
-                <param name="max_velocity">1.0</param>
-                <param name="min_velocity">-1.0</param>
-            </joint>
-            <joint name="joint2">
-                <command_interface name="position"/>
-                <state_interface name="position"/>
-                <state_interface name="velocity"/>
-                <param name="can_id">0x61</param>
-                <param name="gear_ratio">101.0</param>
-                <param name="position_offset">188D6</param>
-                <param name="max_current">22000</param>
-                <param name="min_current">-22000</param>
-                <param name="position_p">5000</param>
-                <param name="position_d">450</param>
-                <param name="velocity_p">550</param>
-                <param name="velocity_i">250</param>
-                <param name="max_velocity">1.0</param>
-                <param name="min_velocity">-1.0</param>
-            </joint>
-            <joint name="joint3">
-                <command_interface name="position"/>
-                <state_interface name="position"/>
-                <state_interface name="velocity"/>
-                <param name="can_id">0x62</param>
-                <param name="gear_ratio">101.0</param>
-                <param name="position_offset">8052</param>
-                <param name="max_current">22000</param>
-                <param name="min_current">-22000</param>
-                <param name="position_p">4600</param>
-                <param name="position_d">400</param>
-                <param name="velocity_p">450</param>
-                <param name="velocity_i">220</param>
-                <param name="max_velocity">1.0</param>
-                <param name="min_velocity">-1.0</param>
-            </joint>
-            <joint name="joint4">
-                <command_interface name="position"/>
-                <state_interface name="position"/>
-                <state_interface name="velocity"/>
-                <param name="can_id">0x63</param>
-                <param name="gear_ratio">121.0</param>
-                <param name="position_offset">28F7</param>
-                <param name="max_current">13000</param>
-                <param name="min_current">-13000</param>
-                <param name="position_p">5200</param>
-                <param name="position_d">500</param>
-                <param name="velocity_p">1250</param>
-                <param name="velocity_i">1500</param>
-                <param name="max_velocity">10.0</param>
-                <param name="min_velocity">-10.0</param>
-            </joint>
-        </ros2_control>
-    </xacro:macro>
+	<xacro:macro name="fold_elevator_ros2_control" params="name sim can_interface desired_config_update_rate">
+		<ros2_control name="fold_elevator" type="system">
+		<hardware>
+			<xacro:if value="${sim}">
+			<plugin>mock_components/GenericSystem</plugin>
+			</xacro:if>
+			<xacro:unless value="${sim}">
+			<plugin>fold_elevator_hardware_interface/FoldElevatorHardwareInterface</plugin>
+			<param name="can_interface">${can_interface}</param>
+			<param name="desired_config_update_rate">${desired_config_update_rate}</param>
+			</xacro:unless>
+		</hardware>
+		<joint name="joint1">
+			<command_interface name="position"/>
+			<state_interface name="position"/>
+			<state_interface name="velocity"/>
+			<param name="can_id">0x60</param>
+			<param name="gear_ratio">101.0</param>
+			<param name="position_offset">A0CC</param>
+			<param name="max_current">22000</param>
+			<param name="min_current">-22000</param>
+			<param name="position_p">5000</param>
+			<param name="position_d">0</param>
+			<param name="velocity_p">300</param>
+			<param name="velocity_i">250</param>
+			<param name="max_velocity">1.0</param>
+			<param name="min_velocity">-1.0</param>
+		</joint>
+		<joint name="joint2">
+			<command_interface name="position"/>
+			<state_interface name="position"/>
+			<state_interface name="velocity"/>
+			<param name="can_id">0x61</param>
+			<param name="gear_ratio">101.0</param>
+			<param name="position_offset">188D6</param>
+			<param name="max_current">22000</param>
+			<param name="min_current">-22000</param>
+			<param name="position_p">4000</param>
+			<param name="position_d">0</param>
+			<param name="velocity_p">90</param>
+			<param name="velocity_i">200</param>
+			<param name="max_velocity">1.0</param>
+			<param name="min_velocity">-1.0</param>
+		</joint>
+		<joint name="joint3">
+			<command_interface name="position"/>
+			<state_interface name="position"/>
+			<state_interface name="velocity"/>
+			<param name="can_id">0x62</param>
+			<param name="gear_ratio">101.0</param>
+			<param name="position_offset">8052</param>
+			<param name="max_current">22000</param>
+			<param name="min_current">-22000</param>
+			<param name="position_p">4600</param>
+			<param name="position_d">0</param>
+			<param name="velocity_p">300</param>
+			<param name="velocity_i">250</param>
+			<param name="max_velocity">1.0</param>
+			<param name="min_velocity">-1.0</param>
+		</joint>
+		<joint name="joint4">
+			<command_interface name="position"/>
+			<state_interface name="position"/>
+			<state_interface name="velocity"/>
+			<param name="can_id">0x63</param>
+			<param name="gear_ratio">121.0</param>
+			<param name="position_offset">28F7</param>
+			<param name="max_current">13000</param>
+			<param name="min_current">-13000</param>
+			<param name="position_p">5200</param>
+			<param name="position_d">0</param>
+			<param name="velocity_p">1250</param>
+			<param name="velocity_i">1500</param>
+			<param name="max_velocity">10.0</param>
+			<param name="min_velocity">-10.0</param>
+		</joint>
+		</ros2_control>
+	</xacro:macro>
 </robot>

Commit message: updated camera lifecycle

File: src/fold_elevator/fold_elevator_configure/config/fold_elevator.ros2_control.xacro (robot description, xacro)
@@ -21,6 +21,6 @@
                 <param name="max_current">22000</param>
                 <param name="min_current">-22000</param>
-                <param name="position_p">4200</param>
-                <param name="position_d">500</param>
+                <param name="position_p">5000</param>
+                <param name="position_d">450</param>
                 <param name="velocity_p">550</param>
                 <param name="velocity_i">250</param>
@@ -37,6 +37,6 @@
                 <param name="max_current">22000</param>
                 <param name="min_current">-22000</param>
-                <param name="position_p">4200</param>
-                <param name="position_d">400</param>
+                <param name="position_p">5000</param>
+                <param name="position_d">450</param>
                 <param name="velocity_p">550</param>
                 <param name="velocity_i">250</param>
@@ -53,5 +53,5 @@
                 <param name="max_current">22000</param>
                 <param name="min_current">-22000</param>
-                <param name="position_p">4000</param>
+                <param name="position_p">4600</param>
                 <param name="position_d">400</param>
                 <param name="velocity_p">450</param>
@@ -69,10 +69,10 @@
                 <param name="max_current">13000</param>
                 <param name="min_current">-13000</param>
-                <param name="position_p">2000</param>
-                <param name="position_d">600</param>
-                <param name="velocity_p">500</param>
-                <param name="velocity_i">250</param>
-                <param name="max_velocity">1.0</param>
-                <param name="min_velocity">-1.0</param>
+                <param name="position_p">5200</param>
+                <param name="position_d">500</param>
+                <param name="velocity_p">1250</param>
+                <param name="velocity_i">1500</param>
+                <param name="max_velocity">10.0</param>
+                <param name="min_velocity">-10.0</param>
             </joint>
         </ros2_control>

File: src/robostore_bringup/urdf/table.urdf.xacro (robot description, xacro)
@@ -33,8 +33,8 @@
     </xacro:place_location>
     <xacro:place_location parent="${name}_${id}_base_link" prefix="${name}_${id}" index="2">
-      <origin xyz="0.5 0.15 ${table_height}" rpy="0 0 0"/>
+      <origin xyz="0.55 0.15 ${table_height}" rpy="0 0 0"/>
     </xacro:place_location>
     <xacro:place_location parent="${name}_${id}_base_link" prefix="${name}_${id}" index="3">
-      <origin xyz="0.6 0.15 ${table_height}" rpy="0 0 0"/>
+      <origin xyz="0.7 0.15 ${table_height}" rpy="0 0 0"/>
     </xacro:place_location>
     <xacro:place_location parent="${name}_${id}_base_link" prefix="${name}_${id}" index="4">
@@ -42,8 +42,8 @@
     </xacro:place_location>
     <xacro:place_location parent="${name}_${id}_base_link" prefix="${name}_${id}" index="5">
-      <origin xyz="0.5 0.05 ${table_height}" rpy="0 0 0"/>
+      <origin xyz="0.55 0.05 ${table_height}" rpy="0 0 0"/>
     </xacro:place_location>
     <xacro:place_location parent="${name}_${id}_base_link" prefix="${name}_${id}" index="6">
-      <origin xyz="0.6 0.05 ${table_height}" rpy="0 0 0"/>
+      <origin xyz="0.7 0.05 ${table_height}" rpy="0 0 0"/>
     </xacro:place_location>
   </xacro:macro>
